File: audio_pipeline.sch (KiCad schematic (older format))
At the start: 13 parts, among them P1 CONN_4, P2 CONN_4, P3 CONN_4, P4 CONN_4, P5 CONN_4, U5 MAX4582, U6 DS1882, U8 RC4580

Commit message: Adding part numbers for everything, for BOM preparation.
Parts:
- C4, C6, C7, C8, C9: Digikey (none) -> 445-5122-1-ND
- P1, P2, P3, P4, P5: Digikey (none) -> WM4926-ND
- U5: Digikey (none) -> MAX4582CSE+-ND
- U6: Digikey (none) -> DS1882Z-050+-ND
- U8: Digikey (none) -> 296-15367-1-ND
Changed lines of the file:
@@
-EESchema Schematic File Version 2  date 8/3/2012 1:01:40 PM
+EESchema Schematic File Version 2  date 8/3/2012 4:17:04 PM
 LIBS:atmel
 LIBS:device
@@
 F 0 "C7" H 3500 5650 50  0000 L CNN
 F 1 "0.1u" H 3500 5450 50  0000 L CNN
+F 4 "445-5122-1-ND" H 3450 5550 60  0001 C CNN "Digikey"
 	1    3450 5550
 	1    0    0    -1
@@
 F 0 "C4" H 1950 4150 50  0000 L CNN
 F 1 "0.1u" H 1950 3950 50  0000 L CNN
+F 4 "445-5122-1-ND" H 1900 4050 60  0001 C CNN "Digikey"
 	1    1900 4050
 	1    0    0    -1
@@
 F 0 "C6" H 2400 4150 50  0000 L CNN
 F 1 "0.1u" H 2400 3950 50  0000 L CNN
+F 4 "445-5122-1-ND" H 2350 4050 60  0001 C CNN "Digikey"
 	1    2350 4050
 	1    0    0    -1
@@
 F 0 "C9" H 4450 6700 50  0000 L CNN
 F 1 "0.1u" H 4450 6500 50  0000 L CNN
+F 4 "445-5122-1-ND" H 4400 6600 60  0001 C CNN "Digikey"
 	1    4400 6600
 	1    0    0    -1
@@
 F 2 "MODULE" H 4900 5800 50  0001 C CNN
 F 3 "DOCUMENTATION" H 5500 6800 50  0001 C CNN
+F 4 "296-15367-1-ND" H 5100 6300 60  0001 C CNN "Digikey"
 	1    5100 6300
 	1    0    0    -1
@@
 F 0 "C8" H 4450 6100 50  0000 L CNN
 F 1 "0.1u" H 4450 5900 50  0000 L CNN
+F 4 "445-5122-1-ND" H 4400 6000 60  0001 C CNN "Digikey"
 	1    4400 6000
 	1    0    0    -1
@@
 F 0 "P5" V 7850 6450 50  0000 C CNN
 F 1 "CONN_4" V 7950 6450 50  0000 C CNN
+F 4 "WM4926-ND" H 7900 6450 60  0001 C CNN "Digikey"
 	1    7900 6450
 	1    0    0    -1
@@
 F 0 "P4" V 6800 1000 50  0000 C CNN
 F 1 "CONN_4" V 6900 1000 50  0000 C CNN
+F 4 "WM4926-ND" H 6850 1000 60  0001 C CNN "Digikey"
 	1    6850 1000
 	1    0    0    -1
@@
 F 0 "P3" V 6100 1000 50  0000 C CNN
 F 1 "CONN_4" V 6200 1000 50  0000 C CNN
+F 4 "WM4926-ND" H 6150 1000 60  0001 C CNN "Digikey"
 	1    6150 1000
 	1    0    0    -1
@@
 F 0 "P2" V 5450 1000 50  0000 C CNN
 F 1 "CONN_4" V 5550 1000 50  0000 C CNN
+F 4 "WM4926-ND" H 5500 1000 60  0001 C CNN "Digikey"
 	1    5500 1000
 	1    0    0    -1
@@
 F 0 "P1" V 4750 1000 50  0000 C CNN
 F 1 "CONN_4" V 4850 1000 50  0000 C CNN
+F 4 "WM4926-ND" H 4800 1000 60  0001 C CNN "Digikey"
 	1    4800 1000
 	1    0    0    -1
@@
 F 1 "MAX4582" H 3300 2450 50  0000 C CNN
 F 2 "MODULE" H 3300 2350 50  0001 C CNN
+F 4 "MAX4582CSE+-ND" H 3300 2350 60  0001 C CNN "Digikey"
 	1    3300 2350
 	1    0    0    -1
@@
 F 1 "DS1882" H 4050 4100 50  0000 C CNN
 F 2 "SOIC16" H 3250 4100 50  0001 C CNN
+F 4 "DS1882Z-050+-ND" H 3650 4600 60  0001 C CNN "Digikey"
 	1    3650 4600
 	1    0    0    -1
